File: USB DUINO MINER ch340/USB_MINER_CH340_c2.brd (EAGLE design)
At the start: 37.8 x 22.9 mm, 16 parts, among them J2 USB_A_PTH_MALE, U1 ATMEGA328P_TQFP, U2 CH340G, Y1 16MHZ, Y2 12MHz

Commit message: Revisi board ch340
Parts:
- moved C1 14.8 mm to (24.8, 20.3)
- moved R4 12.9 mm to (21.8, 14.1), turned to 270 degrees
- moved R3 11.6 mm to (23.7, 14.1), turned to 270 degrees
- moved Y2 11.4 mm to (17.8, 8.89), turned to 180 degrees
- moved L 8.28 mm to (24.9, 3.68), turned to 90 degrees
- moved R5 8.18 mm to (24.9, 6.22)
- moved R6 5.18 mm to (26.7, 11.4), turned to 0 degrees
- moved S1 4.20 mm to (26.7, 15.9)
- moved U2 3.86 mm to (15.2, 15.9), turned to 0 degrees
- moved ISP1 3.82 mm to (31.9, 5.71), flipped to the top, turned to 0 degrees
- moved U1 2.69 mm to (19.1, 12.1)
- moved Y1 2.29 mm to (9.53, 11.4)
- moved D1 0.64 mm to (17.8, 3.17)
Routing:
- net +5V: track 78.3 -> 0.30 mm, vias 1 -> 0
- net RESET: track 45.6 -> 12.0 mm
- net MOSI: track 14.3 -> 0.00 mm
- net D13/SCK: track 10.9 -> 0.00 mm
- net N$1: track 4.29 -> 13.9 mm
- net TX: track 3.39 -> 11.1 mm
- net N$13: track 13.8 -> 7.38 mm
- net N$2: track 10.4 -> 5.08 mm
- net N$14: track 5.26 -> 10.2 mm
- net MISO: track 4.93 -> 0.00 mm
- net N$12: track 7.51 -> 11.8 mm
- net D+: track 10.9 -> 14.6 mm
- net N$3: track 7.08 -> 9.14 mm
- net N$10: track 8.00 -> 6.33 mm
- net N$7: track 4.11 -> 2.62 mm
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