File: USB DUINO MINER ch340/USB_MINER_CH340_c.sch (EAGLE design)
At the start: 16 parts, among them J2 USB_A_PTH_MALE, U1 ATMEGA328P_TQFP, U2 CH340G, Y1 16MHZ, Y2 12MHz

Commit message: Revisi board ch340
Connections:
- removed net SCK: ISP1.SCK
- net D13/SCK: now also ISP1.SCK
- net MISO: now also U1.PB4(CIPO)
- net MOSI: now also U1.PB3(COPI/OC2)
Changed lines of the file:
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@@
 <clearance class="2" value="0.4064"/>
+</class>
+<class number="3" name="smds" width="0" drill="0">
 </class>
 </classes>
@@
 <wire x1="139.7" y1="177.8" x2="147.32" y2="177.8" width="0.1524" layer="91"/>
 <wire x1="147.32" y1="177.8" x2="147.32" y2="162.56" width="0.1524" layer="91"/>
+<label x="147.32" y="165.1" size="1.778" layer="95" rot="R90"/>
+</segment>
+<segment>
+<pinref part="ISP1" gate="G$1" pin="SCK"/>
+<wire x1="83.82" y1="124.46" x2="76.2" y2="124.46" width="0.1524" layer="91"/>
+<label x="76.2" y="124.46" size="1.778" layer="95"/>
 </segment>
 </net>
@@
 </segment>
 </net>
-<net name="N$10" class="2">
+<net name="N$10" class="3">
 <segment>
 <pinref part="U1" gate="U1" pin="PB7(XTAL2/TOSC2)"/>
@@
 <label x="114.3" y="124.46" size="1.778" layer="95"/>
 </segment>
+<segment>
+<pinref part="U1" gate="U1" pin="PB3(COPI/OC2)"/>
+<wire x1="139.7" y1="182.88" x2="147.32" y2="182.88" width="0.1524" layer="91"/>
+<label x="144.78" y="182.88" size="1.778" layer="95"/>
+</segment>
 </net>
 <net name="MISO" class="0">
@@
 <label x="76.2" y="127" size="1.778" layer="95"/>
 </segment>
-</net>
-<net name="SCK" class="0">
-<segment>
-<pinref part="ISP1" gate="G$1" pin="SCK"/>
-<wire x1="83.82" y1="124.46" x2="76.2" y2="124.46" width="0.1524" layer="91"/>
-<label x="76.2" y="124.46" size="1.778" layer="95"/>
-</segment>
-</net>
+<segment>
+<pinref part="U1" gate="U1" pin="PB4(CIPO)"/>
+<wire x1="139.7" y1="180.34" x2="147.32" y2="180.34" width="0.1524" layer="91"/>
+<label x="144.78" y="180.34" size="1.778" layer="95"/>
+</segment>
+</net>

Commit message: update part
ubah part dengan ukuran 0603 menjadi 0805
Parts:
- removed C1: 100nF, SparkFun-Capacitors:10NF-0603-50V-10%
- added C6: 100nF, rcl:C-EUC0805K
- C3: device Condensatori:0015_100NF_0603 -> rcl:C-EUC0805K
- R3, R4, R5, R6: device SparkFun-Resistors:1KOHM-0603-1/10W-1% -> rcl:R-US_R0805
Connections:
- net COM: now also C6.2; no longer C3.2
- net N$14: now also C3.2; no longer C1.2
- net RESET: now also C3.1; no longer C1.1
- net VUSB: now also C6.1; no longer C3.1
Other:
- moved on the sheet: C3
